Commit message: train working

File: robot_model/draco/draco_modified.urdf (robot description, URDF)
Before this commit: robot draco, 40 links, 39 joints
Links:
- link l_knee_fe_ld: geometry collision sphere radius=0.055; collision sphere radius=0.065
- link r_knee_fe_ld: geometry collision sphere radius=0.055; collision sphere radius=0.065
